File: hardware/pcb/c3/tune-button-c3.kicad_pcb (KiCad board)
At the start: 2 copper layers, 46 x 69.5 mm, 39 parts, among them J1 USB-C, J2 LiPo, Q1 AO3401A, SW1 MX switch, SW2 MX switch, SW3 MX switch, SW4 MX switch, SW5 RESET, SW6 BOOT, U1 ESP32-C3-WROOM-02-N4, U2 SRV05-4, U3 TP4054, U4 MCP1700-3.3

Commit message: pcb (c3): power-path fixes from simulation
- SRV05-4 rail on 3V3, not VBUS: on battery the D+ pull-up leaked onto VBUS (2.6 V simulated)
  and half turned off the battery FET.
- 1 ohm in series with the charger's input capacitor: plug-in ringing peaked near 7 V, past the
  regulator's 6.5 V limit.
- R5 100k -> 10k: Q1 turns back on ~3 ms after unplugging rather than ~15 ms, and stays on
  against D2's leakage when warm.
Parts:
- added R13: 1, Resistor_SMD:R_0603_1608Metric, F.Cu at (30.4, 16.5)
- R5: value 100k -> 10k
Connections:
- C1 pad 1: VBUS -> VBUS_C
- U2 pad 5: VBUS -> 3V3
Routing:
- net 3V3: track 52.4 -> 103.7 mm, vias 3 -> 2
- net VBAT: track 82.3 -> 53.0 mm
- net LED_A: track 41.8 -> 18.9 mm
- net VBUS: track 94.3 -> 115.2 mm
- net K3: track 67.1 -> 49.1 mm
- net K1: track 24.3 -> 34.9 mm
- net K4: track 52.0 -> 62.5 mm, vias 1 -> 3
- net USB_DP: track 72.0 -> 61.8 mm, vias 2 -> 4
- net IO9: track 21.0 -> 29.6 mm
- net EN: track 30.1 -> 37.5 mm, vias 0 -> 3
- net STAT: track 14.8 -> 9.05 mm
- net USB_DN: track 59.5 -> 64.4 mm, vias 4 -> 7
- net CHG_A: track 8.99 -> 12.8 mm
- net CC2: track 11.2 -> 7.69 mm, vias 2 -> 0
- net VBUS_C: track 0.00 -> 2.76 mm
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
Commit message: pcb (c3): RT9080 600 mA regulator
Covers Wi-Fi's ~350 mA transmit peaks (current limit >= 610 mA, 2 uA quiescent); SOT-23-5 with the
AP2112K symbol's pinout, EN tied on. JLC CPL rotation +270, from JLC's own footprint.
Parts:
- U4: value MCP1700-3.3 -> RT9080-3.3; footprint Package_TO_SOT_SMD:SOT-23 -> Package_TO_SOT_SMD:SOT-23-5
Connections:
- U4 pad 1: GND -> VSYS
- U4 pad 2: 3V3 -> GND
Routing:
- net USB_DP: track 61.8 -> 84.0 mm
- net K3: track 49.1 -> 68.9 mm
- net VBAT_SENSE: track 28.5 -> 48.0 mm, vias 0 -> 2
- net PROG: track 4.10 -> 16.8 mm, vias 0 -> 2
- net K4: track 62.5 -> 53.6 mm, vias 3 -> 1
- net IO9: track 29.6 -> 21.1 mm
- net 3V3: track 103.7 -> 96.2 mm, vias 2 -> 3
- net EN: track 37.5 -> 31.7 mm, vias 3 -> 0
- net CHG_A: track 12.8 -> 8.30 mm
- net VSYS: track 19.2 -> 23.4 mm, vias 0 -> 2
- net TXD: track 38.6 -> 34.8 mm, vias 2 -> 0
- net VBAT: track 53.0 -> 49.4 mm
- net STAT: track 9.05 -> 5.94 mm
- net GND: track 47.1 -> 44.8 mm, vias 138 -> 135
- net K1: track 34.9 -> 32.7 mm
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