File: hardware/pcb/c3/tune-button-c3.kicad_sch (KiCad schematic)
At the start: 35 parts, among them J1 USB-C, J2 LiPo, Q1 AO3401A, SW1 MX switch, SW2 MX switch, SW3 MX switch, SW4 MX switch, SW5 RESET, SW6 BOOT, U1 ESP32-C3-WROOM-02-N4, U2 USBLC6-2SC6, U3 MCP73831-2, U4 MCP1700-3302E

Commit message: C3 PCB: JLC Basic/Preferred parts where a drop-in exists, LCSC numbers, JLC BOM and CPL
TP4054 for MCP73831, XC6206 for MCP1700 and SRV05-4 for USBLC6-2SC6, each with the same footprint
and pinout. Every assembled part carries its LCSC number; the build writes JLC-format BOM and
placement files listing only those parts. Only the module, USB-C and JST sockets remain Extended.
Parts:
- C1, C2: LCSC (none) -> C19666
- C3, C6: LCSC (none) -> C15849
- C4: LCSC (none) -> C45783
- C5, C7: LCSC (none) -> C14663
- D1, D3: LCSC (none) -> C2286
- D2: LCSC (none) -> C191023
- J1: LCSC (none) -> C165948
- J2: LCSC (none) -> C295747
- Q1: LCSC (none) -> C15127
- R1, R2: LCSC (none) -> C23186
- R10, R11: LCSC (none) -> C22961
- R12, R4: LCSC (none) -> C21190
- R3: LCSC (none) -> C23162
- R5: LCSC (none) -> C25803
- R6, R7, R9: LCSC (none) -> C25804
- SW5, SW6: LCSC (none) -> C318884; MPN XKB TS-1187A -> XKB TS-1187A-B-A-B
- U1: LCSC (none) -> C2934560
- U2: value USBLC6-2SC6 -> SRV05-4; symbol Power_Protection:USBLC6-2SC6 -> Power_Protection:SRV05-4; LCSC (none) -> C85364; MPN USBLC6-2SC6 -> SRV05-4-P-T7
- U3: value MCP73831-2 -> TP4054; symbol Battery_Management:MCP73831-2-OT -> Battery_Management:LTC4054ES5-4.2; LCSC (none) -> C32574; MPN MCP73831T-2ACI/OT -> TP4054-42-SOT25R
- U4: value MCP1700-3302E -> XC6206P332MR; symbol Regulator_Linear:MCP1700x-330xxTT -> Regulator_Linear:XC6206PxxxMR; LCSC (none) -> C5446; MPN MCP1700T-3302E/TT -> XC6206P332MR-G
Other:
- moved on the sheet: U3

Commit message: C3 PCB: switches and LEDs on the back, electronics on the front, EdgeCoil mark on the key side
The MX switches mount on the back (mirrored so K1 is still top left from the key side), and only
their leads and posts need room on the front, guarded by part-free rule areas. That lets the keys
sit behind the electronics: the board is 69.5 mm long instead of 80.5. The two LEDs move to the key
side as hand-soldered 0805s; the battery socket and UART pads sit between the key rows. The key side
carries the mark, the board name and LED labels; part labels are placed per side and kept off the
antenna notch.
Parts:
- D1, D3: footprint LED_SMD:LED_0603_1608Metric -> LED_SMD:LED_0805_2012Metric; LCSC C2286 -> (none)
Changed lines of the file:
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@@
 			(effects (font (size 1.27 1.27)))
 		)
-		(property "Footprint" "LED_SMD:LED_0603_1608Metric"
+		(property "Footprint" "LED_SMD:LED_0805_2012Metric"
 			(at 116.84 264.16 0)
 			(effects (font (size 1.27 1.27)) (hide yes))
@@
 		(property "Datasheet" ""
 			(at 116.84 259.08 0)
-			(effects (font (size 1.27 1.27)) (hide yes))
-		)
-		(property "LCSC" "C2286"
-			(at 116.84 269.24 0)
 			(effects (font (size 1.27 1.27)) (hide yes))
 		)
@@
 			(effects (font (size 1.27 1.27)))
 		)
-		(property "Footprint" "LED_SMD:LED_0603_1608Metric"
+		(property "Footprint" "LED_SMD:LED_0805_2012Metric"
 			(at 193.04 86.36 0)
 			(effects (font (size 1.27 1.27)) (hide yes))
@@
 			(effects (font (size 1.27 1.27)) (hide yes))
 		)
-		(property "LCSC" "C2286"
-			(at 193.04 91.44 0)
-			(effects (font (size 1.27 1.27)) (hide yes))
-		)

Commit message: pcb: MCP1700 regulator, edgecoil.dev on the silkscreen, mark under its own licence
The EdgeCoil mark, name and URL are all rights reserved and outside CERN-OHL-S; derivatives must
remove them. The C3 board's regulator goes back to the 250 mA MCP1700 (C39051, Extended).
Parts:
- U4: value XC6206P332MR -> MCP1700-3.3; symbol Regulator_Linear:XC6206PxxxMR -> Regulator_Linear:MCP1700x-330xxTT; LCSC C5446 -> C39051; MPN XC6206P332MR-G -> MCP1700T-3302E/TT
Changed lines of the file:
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@@
 	)
 	(symbol
-		(lib_id "Regulator_Linear:XC6206PxxxMR")
+		(lib_id "Regulator_Linear:MCP1700x-330xxTT")
 		(at 116.84 60.96 0)
 		(unit 1)
@@
 			(effects (font (size 1.27 1.27)))
 		)
-		(property "Value" "XC6206P332MR"
+		(property "Value" "MCP1700-3.3"
 			(at 116.84 63.5 0)
 			(effects (font (size 1.27 1.27)))
@@
 			(effects (font (size 1.27 1.27)) (hide yes))
 		)
-		(property "MPN" "XC6206P332MR-G"
+		(property "MPN" "MCP1700T-3302E/TT"
 			(at 116.84 68.58 0)
 			(effects (font (size 1.27 1.27)) (hide yes))
 		)
-		(property "LCSC" "C5446"
+		(property "LCSC" "C39051"
 			(at 116.84 71.12 0)
 			(effects (font (size 1.27 1.27)) (hide yes))

Commit message: pcb (c3): power-path fixes from simulation
- SRV05-4 rail on 3V3, not VBUS: on battery the D+ pull-up leaked onto VBUS (2.6 V simulated)
  and half turned off the battery FET.
- 1 ohm in series with the charger's input capacitor: plug-in ringing peaked near 7 V, past the
  regulator's 6.5 V limit.
- R5 100k -> 10k: Q1 turns back on ~3 ms after unplugging rather than ~15 ms, and stays on
  against D2's leakage when warm.
Parts:
- added R13: 1, Resistor_SMD:R_0603_1608Metric, symbol Device:R
- R5: value 100k -> 10k; LCSC C25803 -> C25804
Connections:
- net 3V3: now also U2.5 (VP)
- net VBUS: now also R13.1; no longer C1.1, U2.5 (VP)
- new net VBUS_C: C1.1, R13.2
Other:
- moved on the sheet: R2, R3, R4, R5, R6, R7, R9, SW1, SW2, SW3, SW4, SW5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

Commit message: pcb (c3): RT9080 600 mA regulator
Covers Wi-Fi's ~350 mA transmit peaks (current limit >= 610 mA, 2 uA quiescent); SOT-23-5 with the
AP2112K symbol's pinout, EN tied on. JLC CPL rotation +270, from JLC's own footprint.
Parts:
- U4: value MCP1700-3.3 -> RT9080-3.3; footprint Package_TO_SOT_SMD:SOT-23 -> Package_TO_SOT_SMD:SOT-23-5; symbol Regulator_Linear:MCP1700x-330xxTT -> Regulator_Linear:AP2112K-3.3; LCSC C39051 -> C841192; MPN MCP1700T-3302E/TT -> RT9080-33GJ5
Connections:
- net 3V3: now also U4.5 (VOUT); no longer U4.2 (VO)
- net GND: now also U4.2 (GND); no longer U4.1 (GND)
- net VSYS: now also U4.1 (VIN)
- no-connect marks 4 -> 5
Other:
- moved on the sheet: C6, C7, D1, D2, D3, Q1, R1, R10, R11, R12, R13, R2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

Commit message: pcb (c3): fixes from the second simulation pass
- C1 4.7u -> 10u 0805 (C15850, Basic): with R13, plug-in ringing on low-resistance cables peaks
  around 5.6 V instead of 6.1 V (RT9080 absolute max 6.5 V).
- D4, a 1N5819WS across Q1: in the ~3-5 ms after unplugging, before Q1 turns on, the cell feeds
  VSYS through 0.35 V rather than the body diode's 0.6 V, so a Wi-Fi burst there stays above
  brown-out at a 3.4 V cell.
Parts:
- added D4: 1N5819WS, Diode_SMD:D_SOD-323, symbol Diode:1N5819WS
- C1: value 4.7u -> 10u; footprint Capacitor_SMD:C_0603_1608Metric -> Capacitor_SMD:C_0805_2012Metric; LCSC C19666 -> C15850
Connections:
- net VBAT: now also D4.2 (A)
- net VSYS: now also D4.1 (K)
Other:
- moved on the sheet: Q1, R1, R10, R11, R12, R13, R2, R3, R4, R5, R6, R7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

Commit message: pcb (c3): fixes from the third simulation pass
- C1's damping resistor 1 -> 0.5 ohm (R13 + R14, two Basic 1 ohm): with 1 ohm a stiff 5.5 V
  source and no cell rang VSYS to 6.8 V, past the RT9080's 6.5 V; 0.47 ohm simulated under 6.4 V
  on every cable corner.
- R5 10k -> 3.3k: the bigger C1 had stretched the unplug gap to 13-28 ms; ~5-7 ms again.
- README: D4's hot reverse leakage means the cell's protection board is the overcharge backstop.
Parts:
- added R14: 1, Resistor_SMD:R_0603_1608Metric, symbol Device:R
- R5: value 10k -> 3.3k; LCSC C25804 -> C22978
Connections:
- net VBUS: now also R14.1
- net VBUS_C: now also R14.2
Other:
- moved on the sheet: R2, R3, R4, R5, R6, R7, R9, SW1, SW2, SW3, SW4, SW5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

Commit message: pcb: fixes from the fourth simulation pass
- C3: R13/R14 (plug-in damping) are 1206, not 0603. Each takes a ~35 W,
  ~50 uJ pulse per plug-in from a stiff source, about twice an 0603's
  repetitive pulse rating. Moved flat above U4; C1 nudged down.
- XIAO: D1 is a 1N4148WS, not a BAT54W. A Schottky's reverse leakage
  dragged K4 low while K3 was held, from about 60 C.
- R5 comment: the unplug gap is 5-8 ms, up to ~15 ms at tolerance extremes.
- wiring.md: the divider holds GPIO2 below the high threshold; it doesn't
  select the boot mode on the C3, so that is fine.
- README: the firmware pin map doesn't match either board yet, and a low
  cell sags the C3 rail on Wi-Fi-sized bursts.
Parts:
- R13, R14: footprint Resistor_SMD:R_0603_1608Metric -> Resistor_SMD:R_1206_3216Metric; LCSC C22936 -> C17928
Changed lines of the file:
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@@
 			(effects (font (size 1.27 1.27)))
 		)
-		(property "Footprint" "Resistor_SMD:R_0603_1608Metric"
+		(property "Footprint" "Resistor_SMD:R_1206_3216Metric"
 			(at 269.24 91.44 0)
 			(effects (font (size 1.27 1.27)) (hide yes))
@@
 			(effects (font (size 1.27 1.27)) (hide yes))
 		)
-		(property "LCSC" "C22936"
+		(property "LCSC" "C17928"
 			(at 269.24 96.52 0)
 			(effects (font (size 1.27 1.27)) (hide yes))
@@
 			(effects (font (size 1.27 1.27)))
 		)
-		(property "Footprint" "Resistor_SMD:R_0603_1608Metric"
+		(property "Footprint" "Resistor_SMD:R_1206_3216Metric"
 			(at 269.24 116.84 0)
 			(effects (font (size 1.27 1.27)) (hide yes))
@@
 			(effects (font (size 1.27 1.27)) (hide yes))
 		)
-		(property "LCSC" "C22936"
+		(property "LCSC" "C17928"
 			(at 269.24 121.92 0)
 			(effects (font (size 1.27 1.27)) (hide yes))
