File: hardware/pcb/c3-jst/tune-button-c3-jst.kicad_pcb (KiCad board)
At the start: 2 copper layers, 36 x 50 mm, 40 parts, among them J1 USB-C, J2 LiPo, J3 Buttons, Q1 AO3401A, SW5 RESET, SW6 BOOT, U1 ESP32-C3-WROOM-02-N4, U2 SRV05-4, U3 TP4054, U4 RT9080-3.3, U5 SRV05-4

Commit message: pcb (c3-jst): round-1 audit fixes
JLC CPL rotates the 7-pin JST 180 degrees (JLC draws it pins-down; at 0 it would be
fitted backwards). A ground via 1.7 mm from U5's ground pin, where the ESD return ran
7.7 mm to the nearest via; the J3 pin legend moves to a column on the right so its
keepout leaves room. R15 330 ohm, so a lit button gets about 4 mA. Pin-1 mark clear
of J3's outline; TP1/TP2/U3 labels hidden. README covers the third board: JLC order
notes, rails, mounting, UART ground, the 3.6 V cutoff.
Parts:
- R15: value 1k -> 330
Routing:
- net GND: vias 53 -> 54
Other:
- board text added: "2-5 K1-K4"
- board text added: "J3: 1 GND"
- board text removed: "J3: 1 GND 2-5 K1-K4"
